File: KiCadFiles/FeatheAudio.kicad_sch (KiCad schematic)
At the start: 15 parts, among them J1 Amp Socket 1x7, J3 Conn_01x02_Socket, J4 XIAO LEFT, J5 XIAO RIGHT, J6 Micro_SD_Card, SW1 SW_Push, SW2 SW_Push, SW3 SW_Push

Commit message: Update J5 part number & BOM
Parts:
- J5: Part Number DS1023-16-1*16B81XBX1 work? https://www.tme.eu/en/details/d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 -> 4217-CSHC121-1202A001C1AC-ND https://www.greenconn.com/Uplo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
Changed lines of the file:
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@@
 			)
 		)
-		(property "Part Number" "DS1023-16-1*16B81XBX1 work?  https://www.tme.eu/en/details/ds1023-16-1x16tx1/pin-headers/connfly/ds1023-16-1-16b81xbx1/"
+		(property "Part Number" "  4217-CSHC121-1202A001C1AC-ND   https://www.greenconn.com/Upload/Products/drawing-cshc121.pdf"
 			(at 158.75 110.49 0)
 			(effects
